Commit message: [change] to use unity

File: leo_description/urdf/leo.urdf.xacro (robot description, xacro)
@@ -4,4 +4,8 @@
   <xacro:arg name="mecanum_wheels" default="false"/>
   <xacro:include filename="$(find leo_description)/urdf/macros.xacro"/>
+  <xacro:include filename="$(find leo_description)/ros2_control/leo.ros2_control.xacro"/>
+  <xacro:include filename="$(find leo_description)/unity/leo.unity.xacro"/>
   <xacro:leo mecanum_wheels="$(arg mecanum_wheels)"/>
+  <xacro:leo_ros2_control name="leo"/>
+  <xacro:leo_unity prefix=""/>
 </robot>

File: leo_description/urdf/leo_sim.urdf.xacro (robot description, xacro)
@@ -6,6 +6,10 @@
   <xacro:arg name="mecanum_wheels" default="false"/>
   <xacro:include filename="$(find leo_description)/urdf/macros.xacro"/>
+  <xacro:include filename="$(find leo_description)/ros2_control/leo.ros2_control.xacro"/>
+  <xacro:include filename="$(find leo_description)/unity/leo.unity.xacro"/>
   <xacro:leo_sim robot_ns="$(arg robot_ns)"
                  fixed="$(arg fixed)"
                  mecanum_wheels="$(arg mecanum_wheels)"/>
+  <xacro:leo_ros2_control name="leo"/>
+  <xacro:leo_unity prefix=""/>
 </robot>

File: leo_description/urdf/macros.xacro (robot description, xacro)
@@ -9,4 +9,10 @@
                        imu_translation:='0.0628 -0.0314 -0.0393'
                        mecanum_wheels:=false">
+    <physics_material name="wheel">
+      <friction static="1.0" dynamic="1.0"/>
+    </physics_material>
+    <physics_material name="body">
+      <friction static="0.3" dynamic="0.3"/>
+    </physics_material>
     <xacro:macro name="rocker_link" params="name">
       <link name="${link_prefix}rocker_${name}_link">
@@ -28,4 +34,5 @@
             <mesh filename="package://leo_description/models/Rocker_outline.stl"/>
           </geometry>
+          <physics_material name="body"/>
         </collision>
       </link>
@@ -49,18 +56,15 @@
           <origin xyz="0 0.04485 0" rpy="${pi/2} 0 0"/>
           <geometry>
-            <cylinder radius="0.057" length="0.07"/>
-          </geometry>
+            <cylinder radius="0.0625" length="0.04"/>
+          </geometry>
+          <physics_material name="wheel"/>
         </collision>
+<!--
         <collision>
-          <origin xyz="0 0.04485 0" rpy="${pi/2} 0 0"/>
-          <geometry>
-            <cylinder radius="0.0625" length="0.04"/>
+          <geometry>
+            <mesh filename="package://leo_description/models/Wheel_outline.stl"/>
           </geometry>
         </collision>
-        <collision>
-          <geometry>
-            <mesh filename="package://leo_description/models/Wheel_outline.stl"/>
-          </geometry>
-        </collision>
+-->
       </link>
     </xacro:macro>
@@ -90,4 +94,5 @@
             <mesh filename="package://leo_description/models/Mecanum_wheel_outline.stl"/>
           </geometry>
+          <physics_material name="wheel"/>
         </collision>
       </link>
@@ -95,5 +100,14 @@
     <!-- LINKS -->
     <xacro:if value="${footprint_link}">
-      <link name="${link_prefix}base_footprint"/>
+      <link name="${link_prefix}base_footprint">
+      <inertial>
+        <mass value="0.000001"/>
+        <origin xyz="0 0 0"/>
+        <inertia
+          ixx="0.000001" ixy="0.0" ixz="0.0"
+          iyy="0.000001" iyz="0.0"
+          izz="0.000001"/>
+      </inertial>
+      </link>
     </xacro:if>
     <link name="${link_prefix}base_link">
@@ -115,4 +129,5 @@
           <mesh filename="package://leo_description/models/Chassis_outline.stl"/>
         </geometry>
+        <physics_material name="body"/>
       </collision>
     </link>
@@ -151,4 +166,5 @@
             <cylinder radius="0.0055" length="0.056"/>
           </geometry>
+          <physics_material name="body"/>
         </collision>
       </link>
@@ -178,4 +194,5 @@
       <limit effort="100.0" lower="-0.24" upper="0.24" velocity="100.0"/>
       <dynamics friction="1.0" damping="0.1"/>
+      <unity_drive_api stiffness="30000" damping="0" force_limit="1000000"/>
     </joint>
     <joint name="${joint_prefix}rocker_R_joint" type="${rockers_joint_type}">
@@ -187,4 +204,5 @@
       <dynamics friction="1.0" damping="0.1"/>
       <mimic joint="rocker_L_joint"/>
+      <unity_drive_api stiffness="30000" damping="0" force_limit="1000000"/>
     </joint>
     <joint name="${joint_prefix}wheel_FL_joint" type="continuous">
@@ -200,4 +218,5 @@
       <limit effort="2.0" velocity="6.0"/>
       <dynamics friction="0.3125" damping="0.1"/>
+      <unity_drive_api stiffness="0" damping="30000" force_limit="1000000"/>
     </joint>
     <joint name="${joint_prefix}wheel_RL_joint" type="continuous">
@@ -213,4 +232,5 @@
       <limit effort="2.0" velocity="6.0"/>
       <dynamics friction="0.3125" damping="0.1"/>
+      <unity_drive_api stiffness="0" damping="30000" force_limit="1000000"/>
     </joint>
     <joint name="${joint_prefix}wheel_FR_joint" type="continuous">
@@ -226,4 +246,5 @@
       <limit effort="2.0" velocity="6.0"/>
       <dynamics friction="0.3125" damping="0.1"/>
+      <unity_drive_api stiffness="0" damping="30000" force_limit="1000000"/>
     </joint>
     <joint name="${joint_prefix}wheel_RR_joint" type="continuous">
@@ -239,4 +260,5 @@
       <limit effort="2.0" velocity="6.0"/>
       <dynamics friction="0.3125" damping="0.1"/>
+      <unity_drive_api stiffness="0" damping="30000" force_limit="1000000"/>
     </joint>
     <xacro:if value="${default_antenna}">
@@ -516,5 +538,7 @@
                link_prefix="${link_prefix}"
                mecanum_wheels="${mecanum_wheels}"/>
+    <!--
     <xacro:leo_gazebo robot_ns="${robot_ns}"/>
+    -->
     <xacro:if value="${fixed}">
       <link name="world"/>
